File: pi-top_Template_THT.sch (KiCad schematic (older format))
At the start: 2 parts, among them J1 CONN_02X17, J2 CONN_02X17

Commit message: Added new 3D models
Parts:
- J1: footprint pi-top:3M_951217-4620-XX -> Pin_Headers:Pin_Header_Angled_2x17_Pitch2.00mm
- J2: footprint pi-top:Harwin_M22-6553442R -> Socket_Strips:Socket_Strip_Angled_2x17_Pitch2.00mm
Changed lines of the file:
@@
 F 0 "J1" H 3350 5015 50  0000 C CNN
 F 1 "CONN_02X17" H 3350 4924 50  0000 C CNN
-F 2 "pi-top:3M_951217-4620-XX" H 3350 2900 50  0001 C CNN
+F 2 "Pin_Headers:Pin_Header_Angled_2x17_Pitch2.00mm" H 3350 2900 50  0001 C CNN
 F 3 "" H 3350 2900 50  0001 C CNN
 	1    3350 4000
@@
 F 0 "J2" H 7950 5015 50  0000 C CNN
 F 1 "CONN_02X17" H 7950 4924 50  0000 C CNN
-F 2 "pi-top:Harwin_M22-6553442R" H 7950 2900 50  0001 C CNN
+F 2 "Socket_Strips:Socket_Strip_Angled_2x17_Pitch2.00mm" H 7950 2900 50  0001 C CNN
 F 3 "" H 7950 2900 50  0001 C CNN
 	1    7950 4000
